File: Mechanical_Keyboard.kicad_sch (KiCad schematic)
At the start: 124 parts, among them SW1 MX, SW10 MX, SW11 MX, SW12 MX, SW13 MX, SW14 MX, SW15 MX, SW16 MX, SW17 MX, SW18 MX, SW19 MX, SW2 MX, SW20 MX, SW21 MX, SW22 MX, SW23 MX, SW24 MX, SW25 MX, SW26 MX, SW27 MX, SW28 MX, SW29 MX, SW3 MX, SW30 MX, SW31 MX, SW32 MX, SW33 MX, SW34 MX, SW35 MX, SW36 MX, SW37 MX, SW38 MX, SW39 MX, SW4 MX, SW40 MX, SW41 MX, SW42 MX, SW43 MX, SW44 MX, SW46 MX, SW47 MX, SW48 MX, SW49 MX, SW5 MX, SW51 MX, SW52 MX, SW53 MX, SW54 MX, SW56 MX, SW57 MX, SW58 MX, SW59 MX, SW6 MX, SW61 MX, SW62 MX, SW63 MX, SW64 MX, SW66 MX, SW67 MX, SW7 MX, SW8 MX, SW9 MX

Commit message: Add files via upload
Connections:
- net at D59.1 (K): now also D14.1 (K), D19.1 (K), D24.1 (K), D29.1 (K), D34.1 (K), D39.1 (K), D44.1 (K), D54.1 (K), D9.1 (K), SW59.1
- net at D35.2 (A): now also SW40.2; no longer SW35.2
- net at D22.1 (K): now also D12.1 (K), D17.1 (K), D2.1 (K), D27.1 (K), D32.1 (K), D37.1 (K), D42.1 (K), D47.1 (K), D52.1 (K), D57.1 (K), D62.1 (K), D67.1 (K), D7.1 (K), SW52.1
- net at D66.1 (K): now also D1.1 (K), D11.1 (K), D16.1 (K), D21.1 (K), D26.1 (K), D31.1 (K), D36.1 (K), D41.1 (K), D46.1 (K), D51.1 (K), D56.1 (K), D6.1 (K), D61.1 (K); no longer D67.1 (K)
- net at D25.1 (K): now also D10.1 (K), D15.1 (K), D20.1 (K), D30.1 (K), D35.1 (K), D4.1 (K), D5.1 (K)
- net at D40.2 (A): now also SW35.2; no longer SW40.2
- net at D23.1 (K): now also D13.1 (K), D18.1 (K), D28.1 (K), D3.1 (K), D33.1 (K), D38.1 (K), D43.1 (K), D48.1 (K), D53.1 (K), D58.1 (K), D63.1 (K), D8.1 (K)
- new net: D48.2 (A), SW48.2
- new net: D46.2 (A), SW46.2
- new net: D47.2 (A), SW47.2
- now unconnected: D40.1 (K), D49.2 (A), SW10.1, SW11.1, SW12.1, SW13.1, SW14.1, SW15.1, SW16.1, SW17.1, SW18.1, SW19.1, SW20.1, SW21.1, SW22.1, SW23.1, SW24.1, SW49.2, SW6.1, SW7.1, SW8.1, SW9.1
Other:
- moved on the sheet: D25, SW25, SW30, SW35, SW4, SW40

Commit message: Add files via upload
Connections:
- net at SW33.1: now also SW25.1, SW31.1, SW32.1, SW34.1
- net at SW11.1: now also SW12.1, SW13.1, SW14.1, SW15.1
- net at D12.1 (K), D17.1 (K), D2.1 (K)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: now also SW35.1, SW51.1, SW53.1, SW54.1
- net at SW48.1: now also SW30.1, SW46.1, SW47.1, SW49.1
- net at SW29.1: now also SW26.1, SW27.1, SW28.1
- net at D14.1 (K), D19.1 (K), D24.1 (K)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: no longer SW59.1
- net at SW8.1: now also SW10.1, SW6.1, SW7.1, SW9.1
- net at SW18.1: now also SW16.1, SW17.1, SW19.1, SW20.1
- net at D13.1 (K), D18.1 (K), D23.1 (K)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: now also SW41.1, SW42.1, SW43.1, SW44.1
- net at SW61.1: now also SW40.1, SW62.1, SW63.1, SW64.1
- net at SW66.1: now also SW67.1
- net at SW36.1: now also SW37.1, SW38.1, SW39.1
- net at SW22.1: now also SW21.1, SW23.1, SW24.1
- net at SW57.1: now also SW4.1, SW56.1, SW58.1, SW59.1

Commit message: Add files via upload
Parts:
- added U1: ATmega32U4-A, Package_QFP:TQFP-44_10x10mm_P0.8mm, symbol MCU_Microchip_ATmega:ATmega32U4-A
Connections:
- net at SW25.1, SW31.1, SW32.1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: now also U1.20 (PD2)
- net at SW11.1, SW12.1, SW13.1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: now also U1.26 (PD6)
- net at D1.1 (K), D11.1 (K), D16.1 (K)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: now also U1.28 (PB4)
- net at D12.1 (K), D17.1 (K), D2.1 (K)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: now also U1.11 (PB3), U1.31 (PC6)
- net at SW30.1, SW46.1, SW47.1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: now also U1.32 (PC7)
- net at SW26.1, SW27.1, SW28.1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: now also U1.21 (PD3)
- net at D14.1 (K), D19.1 (K), D24.1 (K)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: now also U1.9 (PB1)
- net at SW10.1, SW6.1, SW7.1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: now also U1.27 (PD7)
- net at D10.1 (K), D15.1 (K), D20.1 (K)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: now also U1.8 (PB0)
- net at SW16.1, SW17.1, SW18.1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: now also U1.22 (PD5)
- net at D13.1 (K), D18.1 (K), D23.1 (K)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: now also U1.10 (PB2), U1.18 (PD0)
- net at SW40.1, SW61.1, SW62.1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: now also U1.30 (PB6)
- net at SW66.1, SW67.1: now also U1.29 (PB5)
- net at SW36.1, SW37.1, SW38.1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: now also U1.19 (PD1)
- net at SW21.1, SW22.1, SW23.1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: now also U1.25 (PD4)
- net at SW1.1, SW2.1, SW3.1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: now also U1.33 (~{HWB}/PE2)
- net at SW4.1, SW56.1, SW57.1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: now also U1.12 (PB7)
- new net: U1.14 (VCC), U1.34 (VCC)
- new net: U1.15 (GND), U1.23 (GND), U1.35 (GND), U1.43 (GND)
- new net: U1.24 (AVCC), U1.44 (AVCC)

Commit message: Add files via upload
lots of research and a little sketch
https://www.reddit.com/r/PrintedCircuitBoard/comments/kvat9d/usb_type_c_with_atmega32u4/
https://www.digikey.com/en/products/detail/gct/USB4110-GF-A/10384547
Parts:
- added J1: USB_C_Receptacle_USB2.0_14P, Connector_USB:USB_C_Receptacle_GCT_USB4085, symbol Connector:USB_C_Receptacle_USB2.0_14P
- added R1, R2: R5.1k, Resistor_SMD:R_1206_3216Metric, symbol Device:R
Connections:
- net at U1.15 (GND), U1.23 (GND), U1.35 (GND)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: now also J1.A1 (GND), J1.A12 (GND), J1.B1 (GND), J1.B12 (GND), J1.S1 (SHIELD), R1.2, R2.2
- net at U1.3 (D-): now also J1.A7 (D-), J1.B7 (D-)
- net at U1.4 (D+): now also J1.A6 (D+), J1.B6 (D+)
- net at U1.7 (VBUS): now also J1.A4 (VBUS), J1.A9 (VBUS), J1.B4 (VBUS), J1.B9 (VBUS)
- new net: J1.B5 (CC2), R1.1
- new net: J1.A5 (CC1), R2.1

Commit message: Add files via upload
Parts:
- D1, D10, D11, D12, D13, D14, D15, D16, D17, D18, D19, D2, D20, D21, D22, D23, D24, D25, D26, D27, D28, D29, D3, D30, D31, D32, D33, D34, D35, D36, D37, D38, D39, D4, D40, D41, D42, D43, D44, D46, D47, D48, D49, D5, D51, D52, D53, D54, D56, D57, D58, D59, D6, D61, D62, D63, D64, D66, D67, D7, D8, D9: footprint (none) -> Diode_SMD:D_SOD-123
- SW1, SW11, SW12, SW13, SW14, SW16, SW17, SW18, SW19, SW20, SW21, SW22, SW23, SW24, SW26, SW27, SW28, SW29, SW31, SW32, SW33, SW34, SW36, SW37, SW38, SW39, SW41, SW42, SW43, SW44, SW46, SW47, SW48, SW49, SW51, SW52, SW53, SW54, SW56, SW57, SW58, SW59, SW6, SW61, SW62, SW66, SW7, SW8: footprint (none) -> Button_Switch_Keyboard:SW_Cherry_MX_1.00u_PCB
- SW10, SW15, SW30, SW35, SW4, SW40, SW5: footprint (none) -> Button_Switch_Keyboard:SW_Cherry_MX_1.25u_PCB
- SW2: footprint (none) -> Button_Switch_Keyboard:SW_Cherry_MX_1.50u_PCB
- SW25: footprint (none) -> Button_Switch_Keyboard:SW_Cherry_MX_6.25u_PCB
- SW3, SW67: footprint (none) -> Button_Switch_Keyboard:SW_Cherry_MX_1.75u_PCB
- SW63, SW9: footprint (none) -> Button_Switch_Keyboard:SW_Cherry_MX_2.00u_PCB
- SW64: footprint (none) -> Button_Switch_Keyboard:SW_Cherry_MX_2.25u_PCB
