File: IceBox.kicad_sch (KiCad schematic)
At the start: 128 parts, among them J1 USB_C_Receptacle_USB2.0_14P, SW1 ,, SW10 2, SW11 w, SW12 s, SW13 z, SW14 OS, SW15 3, SW16 e, SW17 d, SW18 x, SW19 Alt, SW2 tab, SW20 4, SW21 r, SW22 f, SW23 c, SW24 5, SW25 t, SW26 g, SW27 v, SW28 6, SW29 y, SW3 magic, SW30 h, SW31 b, SW32 Space, SW33 7, SW34 u, SW35 j, SW36 n, SW37 8, SW38 i, SW39 k, SW4 Ctrl, SW40 m, SW41 Alt, SW42 9, SW43 o, SW44 l, SW45 ,, SW46 Mute, SW47 0, SW48 p, SW49 ;, SW5 1, SW50 ., SW51 Vol up, SW52 -, SW53 [, SW54 ', SW55 /, SW56 Vol Down, SW57 =, SW58 ], SW59 Enter, SW6 q, SW60 shift, SW61 PrtScreen, SW62 \, SW7 a, SW8 Shift, SW9 Fn, U1 ATmega32U4-A

Commit message: Add files via upload
Connections:
- net at D12.1 (K), D17.1 (K), D22.1 (K)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: no longer SW37.1, SW38.1, SW39.1, SW40.1, U1.18 (PD0)
- net at D13.1 (K), D18.1 (K), D23.1 (K)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: now also D45.1 (K), D60.1 (K)
- net at D11.1 (K), D16.1 (K), D2.1 (K)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: no longer SW46.1, SW47.1, SW48.1, SW49.1, SW50.1, U1.31 (PC6)
- net at SW28.1, SW29.1, SW30.1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: now also SW36.1, U1.27 (PD7); no longer SW31.1, U1.20 (PD2)
- net at SW61.1, SW62.1: now also SW56.1, U1.18 (PD0); no longer U1.29 (PB5)
- net at D1.1 (K), D10.1 (K), D15.1 (K)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: now also U1.12 (PB7); no longer U1.28 (PB4)
- net at SW15.1, SW16.1, SW17.1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: now also SW23.1, U1.30 (PB6); no longer SW18.1, U1.22 (PD5)
- net at SW10.1, SW11.1, SW12.1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: now also SW18.1, U1.31 (PC6); no longer SW13.1, U1.26 (PD6)
- net at D14.1 (K), D19.1 (K), D32.1 (K)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: now also D46.1 (K)
- net at SW1.1, SW2.1, SW3.1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: now also SW8.1
- net at SW52.1, SW53.1, SW54.1: now also SW46.1, SW60.1, U1.20 (PD2); no longer SW51.1, SW55.1, U1.12 (PB7)
- net at SW24.1, SW25.1, SW26.1: now also SW31.1, U1.28 (PB4); no longer SW27.1, U1.21 (PD3)
- net at SW33.1, SW34.1, SW35.1: now also SW40.1, U1.26 (PD6); no longer SW36.1, U1.19 (PD1)
- net at SW42.1, SW43.1, SW44.1: now also SW50.1, U1.22 (PD5); no longer SW41.1, SW45.1, U1.32 (PC7)
- net at SW57.1, SW58.1, SW59.1: now also SW51.1, U1.19 (PD1); no longer SW56.1, SW60.1, U1.30 (PB6)
- net at SW20.1, SW21.1, SW22.1: now also SW27.1, U1.29 (PB5); no longer SW23.1, U1.25 (PD4)
- net at SW5.1, SW6.1, SW7.1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: now also SW13.1, U1.32 (PC7); no longer SW8.1, U1.27 (PD7)
- net at D45.2 (A): now also SW45.2
- new net: SW41.1, SW47.1, SW48.1, SW49.1, SW55.1, U1.21 (PD3)
- new net: SW37.1, SW38.1, SW39.1, SW45.1, U1.25 (PD4)
Other:
- moved on the sheet: D13, D18, D23, D27, D31, D36, D40, D41, D45, D46, D50, D51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
