File: IceBox.kicad_pcb (KiCad board)
At the start: 2 copper layers, 128 parts, among them J1 USB_C_Receptacle_USB2.0_14P, SW1 ,, SW10 2, SW11 w, SW12 s, SW13 z, SW14 OS, SW15 3, SW16 e, SW17 d, SW18 x, SW19 Alt, SW2 tab, SW20 4, SW21 r, SW22 f, SW23 c, SW24 5, SW25 t, SW26 g, SW27 v, SW28 6, SW29 y, SW3 magic, SW30 h, SW31 b, SW32 Space, SW33 7, SW34 u, SW35 j, SW36 n, SW37 8, SW38 i, SW39 k, SW4 Ctrl, SW40 m, SW41 Alt, SW42 9, SW43 o, SW44 l, SW45 ,, SW46 Mute, SW47 0, SW48 p, SW49 ;, SW5 1, SW50 ., SW51 Vol up, SW52 -, SW53 [, SW54 ', SW55 /, SW56 Vol Down, SW57 =, SW58 ], SW59 Enter, SW6 q, SW60 shift, SW61 PrtScreen, SW62 \, SW7 a, SW8 Shift, SW9 Fn, U1 ATmega32U4-A

Commit message: new
Parts:
- moved J1 198.2 mm to (139.5, 30.0), turned to 180 degrees
- moved U1 197.5 mm to (117.2, 35.4), turned to -90 degrees
- moved D5 168.2 mm to (28.1, 60.5), turned to 90 degrees
- moved D1 166.2 mm to (9.58, 60.5), turned to 90 degrees
- moved D42 163.1 mm to (187.6, 62.1), turned to 90 degrees
- moved R2 158.5 mm to (199.5, 23.5)
- moved D15 156.2 mm to (67.6, 63.5), turned to 90 degrees
- moved D33 153.5 mm to (147.6, 62.5), turned to 90 degrees
- moved R1 153.2 mm to (200.3, 25.5)
- moved D43 153.0 mm to (198.6, 81.7), turned to 90 degrees
- moved D2 151.6 mm to (13.1, 79.3), turned to 90 degrees
- moved D24 151.2 mm to (107.6, 62.9), turned to 90 degrees
- moved D6 150.8 mm to (35.6, 79.5), turned to 90 degrees
- moved D10 146.3 mm to (50.2, 63.5), turned to 90 degrees
- moved D44 142.8 mm to (203.1, 99.3), turned to 90 degrees
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Connections:
- D45 pad 1: unconnected-(D45-K-Pad1) -> Net-(D13-K)
- D45 pad 2: unconnected-(D45-A-Pad2) -> Net-(D45-A)
- D46 pad 1: unconnected-(D46-K-Pad1) -> Net-(D14-K)
- SW13 pad 1: Net-(U1-PD6) -> Net-(U1-PD7)
- SW18 pad 1: Net-(U1-PD5) -> Net-(U1-PD6)
- SW23 pad 1: Net-(U1-PD4) -> Net-(U1-PD5)
- SW27 pad 1: Net-(U1-PD3) -> Net-(U1-PD4)
- SW31 pad 1: Net-(U1-PD2) -> Net-(U1-PD3)
- SW36 pad 1: Net-(U1-PD1) -> Net-(U1-PD2)
- SW37 pad 1: Net-(D12-K) -> Net-(U1-PD0)
- SW38 pad 1: Net-(D12-K) -> Net-(U1-PD0)
- SW39 pad 1: Net-(D12-K) -> Net-(U1-PD0)
- SW40 pad 1: Net-(D12-K) -> Net-(U1-PD1)
- SW41 pad 1: Net-(U1-PC7) -> Net-(U1-PC6)
- SW45 pad 1: Net-(U1-PC7) -> Net-(U1-PD0)
- SW45 pad 2: unconnected-(SW45-Pad2) -> Net-(D45-A)
- SW46 pad 1: Net-(D11-K) -> Net-(U1-PB7)
- SW47 pad 1: Net-(D11-K) -> Net-(U1-PC6)
- SW48 pad 1: Net-(D11-K) -> Net-(U1-PC6)
- SW49 pad 1: Net-(D11-K) -> Net-(U1-PC6)
- SW50 pad 1: Net-(D11-K) -> Net-(U1-PC7)
- SW51 pad 1: Net-(U1-PB7) -> Net-(U1-PB6)
- SW55 pad 1: Net-(U1-PB7) -> Net-(U1-PC6)
- SW56 pad 1: Net-(U1-PB6) -> Net-(U1-PB5)
- SW60 pad 1: Net-(U1-PB6) -> Net-(U1-PB7)
- SW8 pad 1: Net-(U1-PD7) -> Net-(U1-~{HWB}/PE2)
- U1 pad 18: Net-(D12-K) -> Net-(U1-PD0)
- U1 pad 31: Net-(D11-K) -> Net-(U1-PC6)

Commit message: Add files via upload
Parts:
- moved D10 2.23 mm to (48.0, 63.5)
Connections:
- D60 pad 1: unconnected-(D60-K-Pad1) -> Net-(D13-K)
Routing:
- net Net-(D14-K): track 0.00 -> 292.0 mm
- net Net-(D11-K): track 0.00 -> 272.3 mm
- net Net-(D1-K): track 0.00 -> 259.4 mm
- net Net-(D12-K): track 0.00 -> 256.2 mm
- net Net-(D13-K): track 0.00 -> 250.9 mm
- net Net-(U1-PD7): track 0.00 -> 93.3 mm
- net Net-(U1-PD6): track 0.00 -> 92.4 mm
- net Net-(U1-PD5): track 0.00 -> 91.1 mm
- net Net-(U1-PD2): track 0.00 -> 91.1 mm
- net Net-(U1-~{HWB}/PE2): track 0.00 -> 89.3 mm
- net Net-(U1-PD3): track 0.00 -> 68.5 mm
- net Net-(U1-PD4): track 0.00 -> 68.3 mm
- net Net-(U1-PD1): track 0.00 -> 24.9 mm
- net Net-(D59-A): track 0.00 -> 16.7 mm
- net Net-(D60-A): track 0.00 -> 13.1 mm
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
Commit message: Add files via upload
Parts:
- moved U1 28.2 mm to (145.0, 40.0), turned to 90 degrees
Routing:
- net Net-(U1-PB5): track 0.00 -> 235.9 mm
- net Net-(U1-PB7): track 0.00 -> 221.0 mm
- net Net-(U1-PB6): track 0.00 -> 219.6 mm
- net Net-(U1-PC7): track 0.00 -> 137.0 mm
- net Net-(U1-PC6): track 0.00 -> 133.5 mm
- net Net-(U1-PD6): track 92.4 -> 194.3 mm
- net Net-(D14-K): track 292.0 -> 371.6 mm
- net Net-(U1-PD0): track 0.00 -> 69.6 mm
- net Net-(U1-PD4): track 68.3 -> 125.9 mm
- net Net-(U1-PD1): track 24.9 -> 71.2 mm
- net Net-(U1-~{HWB}/PE2): track 89.3 -> 118.4 mm
- net Net-(J1-SHIELD): track 0.00 -> 1.19 mm
- net Net-(U1-PD7): track 93.3 -> 94.3 mm

Commit message: Add files via upload
Parts:
- moved J1 129.9 mm to (223.0, 129.5)
- moved U1 125.4 mm to (218.0, 142.0), turned to -90 degrees
- moved R2 112.0 mm to (223.0, 133.0)
- moved D28 110.2 mm to (20.8, 87.7)
- moved D29 110.2 mm to (31.3, 106.5)
- moved D30 110.2 mm to (36.3, 124.5)
- moved D31 110.2 mm to (21.8, 144.7)
- moved D32 110.2 mm to (40.3, 165.6)
- moved D33 110.2 mm to (40.3, 87.7)
- moved D34 110.2 mm to (51.3, 106.8)
- moved D35 110.2 mm to (56.8, 124.7)
- moved D36 110.2 mm to (42.3, 145.2)
- moved D37 110.2 mm to (60.3, 87.7)
- moved D38 110.2 mm to (71.3, 106.8)
- moved D39 110.2 mm to (76.3, 124.7)
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Connections:
- SW10 pad 1: Net-(U1-PD6) -> Net-(U1-PC6)
- SW11 pad 1: Net-(U1-PD6) -> Net-(U1-PC6)
- SW12 pad 1: Net-(U1-PD6) -> Net-(U1-PC6)
- SW13 pad 1: Net-(U1-PD7) -> Net-(U1-PC7)
- SW14 pad 1: Net-(U1-PD6) -> Net-(U1-PC6)
- SW15 pad 1: Net-(U1-PD5) -> Net-(U1-PB6)
- SW16 pad 1: Net-(U1-PD5) -> Net-(U1-PB6)
- SW17 pad 1: Net-(U1-PD5) -> Net-(U1-PB6)
- SW18 pad 1: Net-(U1-PD6) -> Net-(U1-PC6)
- SW19 pad 1: Net-(U1-PD5) -> Net-(U1-PB6)
- SW20 pad 1: Net-(U1-PD4) -> Net-(U1-PB5)
- SW21 pad 1: Net-(U1-PD4) -> Net-(U1-PB5)
- SW22 pad 1: Net-(U1-PD4) -> Net-(U1-PB5)
- SW23 pad 1: Net-(U1-PD5) -> Net-(U1-PB6)
- SW24 pad 1: Net-(U1-PD3) -> Net-(U1-PB4)
- SW25 pad 1: Net-(U1-PD3) -> Net-(U1-PB4)
- SW26 pad 1: Net-(U1-PD3) -> Net-(U1-PB4)
- SW27 pad 1: Net-(U1-PD4) -> Net-(U1-PB5)
- SW28 pad 1: Net-(U1-PD2) -> Net-(U1-PD7)
- SW29 pad 1: Net-(U1-PD2) -> Net-(U1-PD7)
- SW30 pad 1: Net-(U1-PD2) -> Net-(U1-PD7)
- SW31 pad 1: Net-(U1-PD3) -> Net-(U1-PB4)
- SW32 pad 1: Net-(U1-PD2) -> Net-(U1-PD7)
- SW33 pad 1: Net-(U1-PD1) -> Net-(U1-PD6)
- SW34 pad 1: Net-(U1-PD1) -> Net-(U1-PD6)
- SW35 pad 1: Net-(U1-PD1) -> Net-(U1-PD6)
- SW36 pad 1: Net-(U1-PD2) -> Net-(U1-PD7)
- SW37 pad 1: Net-(U1-PD0) -> Net-(U1-PD4)
- SW38 pad 1: Net-(U1-PD0) -> Net-(U1-PD4)
- SW39 pad 1: Net-(U1-PD0) -> Net-(U1-PD4)
- SW40 pad 1: Net-(U1-PD1) -> Net-(U1-PD6)
- SW41 pad 1: Net-(U1-PC6) -> Net-(U1-PD3)
- SW42 pad 1: Net-(U1-PC7) -> Net-(U1-PD5)
- SW43 pad 1: Net-(U1-PC7) -> Net-(U1-PD5)
- SW44 pad 1: Net-(U1-PC7) -> Net-(U1-PD5)
- SW45 pad 1: Net-(U1-PD0) -> Net-(U1-PD4)
- SW46 pad 1: Net-(U1-PB7) -> Net-(U1-PD2)
- SW47 pad 1: Net-(U1-PC6) -> Net-(U1-PD3)
- SW48 pad 1: Net-(U1-PC6) -> Net-(U1-PD3)
- SW49 pad 1: Net-(U1-PC6) -> Net-(U1-PD3)
- SW5 pad 1: Net-(U1-PD7) -> Net-(U1-PC7)
- SW50 pad 1: Net-(U1-PC7) -> Net-(U1-PD5)
- SW51 pad 1: Net-(U1-PB6) -> Net-(U1-PD1)
- SW52 pad 1: Net-(U1-PB7) -> Net-(U1-PD2)
- SW53 pad 1: Net-(U1-PB7) -> Net-(U1-PD2)
- SW54 pad 1: Net-(U1-PB7) -> Net-(U1-PD2)
- SW55 pad 1: Net-(U1-PC6) -> Net-(U1-PD3)
- SW56 pad 1: Net-(U1-PB5) -> Net-(U1-PD0)
- SW57 pad 1: Net-(U1-PB6) -> Net-(U1-PD1)
- SW58 pad 1: Net-(U1-PB6) -> Net-(U1-PD1)
- SW59 pad 1: Net-(U1-PB6) -> Net-(U1-PD1)
- SW6 pad 1: Net-(U1-PD7) -> Net-(U1-PC7)
- SW60 pad 1: Net-(U1-PB7) -> Net-(U1-PD2)
- SW61 pad 1: Net-(U1-PB5) -> Net-(U1-PD0)
- SW62 pad 1: Net-(U1-PB5) -> Net-(U1-PD0)
- SW7 pad 1: Net-(U1-PD7) -> Net-(U1-PC7)
- SW9 pad 1: Net-(U1-PD7) -> Net-(U1-PC7)
- U1 pad 11: Net-(D11-K) -> Net-(D13-K)
- U1 pad 12: Net-(U1-PB7) -> Net-(D14-K)
- U1 pad 28: Net-(D1-K) -> Net-(U1-PB4)
- U1 pad 8: Net-(D14-K) -> Net-(D1-K)
- U1 pad 9: Net-(D13-K) -> Net-(D11-K)
Routing:
- net Net-(U1-~{HWB}/PE2): track 118.4 -> 446.7 mm
- net Net-(U1-PB4): track 0.00 -> 314.4 mm
- net Net-(U1-PC7): track 137.0 -> 418.8 mm
- net Net-(U1-PC6): track 133.5 -> 392.0 mm
- net Net-(U1-PB7): track 221.0 -> 0.00 mm
- net Net-(U1-PD7): track 94.3 -> 286.6 mm
- net Net-(U1-PD3): track 68.5 -> 216.7 mm
- net Net-(U1-PB6): track 219.6 -> 366.5 mm
- net Net-(U1-PD5): track 91.1 -> 233.1 mm
- net Net-(U1-PD4): track 125.9 -> 247.4 mm
- net Net-(U1-PD2): track 91.1 -> 206.7 mm
- net Net-(U1-PB5): track 235.9 -> 337.3 mm
- net Net-(U1-PD1): track 71.2 -> 171.4 mm
- net Net-(U1-PD6): track 194.3 -> 272.1 mm
- net Net-(D1-K): track 259.4 -> 336.7 mm
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Other:
- board outline added: 328 x 116 mm
